File: electronics/pzpre.kicad_pcb (KiCad board)
At the start: 2 copper layers, 54 x 61 mm, 32 parts, among them Q1 2SK3666, U1 LTC1540

Commit message: wip
Parts:
- removed C2: 470p, smd_cap:c_0603
- removed C3: 100n, smd_cap:c_0603
- removed C4: 470n, smd_cap:c_0805
- removed C5: 1u, smd_cap:c_0805
- removed C6: 10u, smd_cap:c_tant_C
- removed D1, D2: 1PS76SB40, diodes:SOD-323
- removed LED1: LED, WL-SMTWSMD
- removed PL1: MOLEX_2_PIN_HEADER, connectors:MOLEX_2_PIN_2_54
- removed R10: 680, R3
- removed R11: 2M4, smd_res:r_0603
- removed R12: 7k5, smd_res:r_0603
- removed R13: 430, smd_res:r_0603
- removed R14: 10, smd_res:r_0603
- removed R4: 6M34, smd_res:r_0603
- removed R5: 10K, smd_res:r_0603
- removed R6: 2k4, smd_res:r_0603
- removed R7: 1M18, smd_res:r_0603
- removed R8: 47k, smd_res:r_0603
- removed R9: 2k4, R3
- removed SK1, SK2: JACK_SOCKET_6_35_STEREO, connectors:JACK_SOCKET_6_35_NEUTRIK_NMJ6HFD2
- removed U1: LTC1540, msop:MSOP8
- added H5: HOLE, aart_holes:PLATED_HOLE_1_5MM, F.Cu at (247.9, 200.3)
- C1: value 10u -> C; footprint smd_cap:c_tant_C -> w_smd_cap:c_0805
- H1, H2, H3, H4: footprint holes:UNPLATED_HOLE_3MM -> aart_holes:PLATED_HOLE_1_5MM
- Q1: footprint smd_trans:sot23 -> w_smd_trans:sot23
- R1: value 6M34 -> R; footprint smd_res:r_0603 -> w_smd_resistors:r_0603
- R2: value 680 -> R; footprint smd_res:r_0603 -> w_smd_resistors:r_0603
- R3: value 3k3 -> R; footprint smd_res:r_0603 -> w_smd_resistors:r_0603
- moved H4 100.9 mm to (250.6, 206.9)
- moved H3 100.0 mm to (252.2, 194.4)
- moved Q1 72.9 mm to (226.4, 202.3)
- moved R3 67.5 mm to (219.9, 195.8)
- moved H2 67.5 mm to (258.0, 204.8)
- moved R1 62.1 mm to (223.9, 190.8), turned to 0 degrees
- moved R2 54.4 mm to (227.9, 187.3)
- moved C1 49.0 mm to (226.9, 197.3), turned to 0 degrees
- moved H1 36.7 mm to (258.2, 199.0)
Connections:
- C1 pad 1: /Vcc -> Net-(C1-Pad1)
- C1 pad 2: 0VA -> Net-(C1-Pad2)
- Q1 pad 2: Net-(C4-Pad1) -> Net-(C1-Pad2)
- R1 pad 2: 0VA -> Net-(H2-Pad1)
- R2 pad 1: Net-(Q1-Pad1) -> Net-(H1-Pad1)
- R2 pad 2: 0VA -> Net-(C1-Pad2)
- R3 pad 1: Net-(LED1-Pad2) -> Net-(Q1-Pad1)
- R3 pad 2: Net-(R3-Pad2) -> Net-(H2-Pad1)
Routing:
- net /Vcc: track 120.7 -> 0.00 mm, vias 1 -> 0
- net Net-(PL1-Pad2): track 81.7 -> 0.00 mm
- net Net-(SK1-Pad2): track 57.9 -> 0.00 mm
- net Net-(C4-Pad2): track 30.3 -> 0.00 mm
- net Net-(C6-Pad1): track 23.7 -> 0.00 mm
- net Net-(R5-Pad1): track 15.6 -> 0.00 mm
- net Net-(LED1-Pad2): track 13.4 -> 0.00 mm, vias 1 -> 0
- net Net-(D1-Pad1): track 13.3 -> 0.00 mm
- net Net-(C4-Pad1): track 12.2 -> 0.00 mm
- net Net-(H5-Pad1): track 10.6 -> 0.00 mm
- net Net-(Q1-Pad1): track 10.4 -> 0.00 mm
- net Net-(R12-Pad1): track 9.20 -> 0.00 mm
- net Net-(R11-Pad1): track 8.57 -> 0.00 mm
- net Net-(R3-Pad2): track 6.46 -> 0.00 mm
- net Net-(R4-Pad2): track 4.26 -> 0.00 mm
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- removed copper zone on B.Cu, net 0VA
- removed copper zone on F.Cu, net 0VA
Other:
- board size 54 x 61 mm -> 24 x 27 mm
- board text removed: "+"
- board text removed: "-"
- board text removed: "FPRE-01"
