File: electronics/pzpre.sch (KiCad schematic (older format))
At the start: 27 parts, among them U1 LTC1540

Commit message: wip
Parts:
- removed C1, C6: 47u, symbol CPol
- removed C3: 100n, symbol C
- removed C5: 1u, symbol C
- removed D1, D2: 1PS76SB40, symbol SCHOTTKY
- removed LED1: LED, ~, symbol LED
- removed PL1: MOLEX_2_PIN_HEADER, symbol MOLEX_2_PIN_HEADER
- removed R11: 2M4, symbol R
- removed R12: 7k5, symbol R
- removed R13: 430, symbol R
- removed R14: 10, symbol R
- removed R4: 6M34, symbol R
- removed R5: 10K, symbol R
- removed R7: 1M18, symbol R
- removed R?: 100, symbol R
- removed SK1, SK2: JACK_SOCKET_6_35_STEREO, symbol JACK_SOCKET_6_35_STEREO
- removed U1: LTC1540, symbol LTC1540
- removed U? (x3): LTC6241HV, symbol LTC6241HV
- added C1: C, w_smd_cap:c_0805, symbol C
- added H5: HOLE, aart_holes:PLATED_HOLE_1_5MM, symbol HOLE
- added Q1: 2SK3666, w_smd_trans:sot23, symbol FET_N
- added R1, R2: R, w_smd_resistors:r_0603, symbol R
- H1, H2, H3, H4: footprint (none) -> aart_holes:PLATED_HOLE_1_5MM
- R3: value 3k3 -> R; footprint (none) -> w_smd_resistors:r_0603
Connections:
- net labels removed: 0VA, GND, VCC, Vcc
- wire segments 54 -> 11
Other:
- note removed: "battery monitor (LED on above 7.5V)"
- moved on the sheet: H1, H2, H3, H4
